File: POV_Bike.kicad_pcb (KiCad board)
At the start: 2 copper layers, 50.8 x 99.1 mm, 24 parts, among them IC1 ATTINY44-P, P1 CONN_6, U1 A1120

Commit message: Melhorias no layout da placa
Routing:
- net N-0000018: track 37.4 -> 40.7 mm
